File: Nixie_clock.kicad_sch (KiCad schematic)
At the start: 29 parts, among them J1 Screw_Terminal_01x02, J2 Screw_Terminal_01x03, U1 74HCT04, U10 TPIC6B595, U11 TPIC6B595, U2 TPIC6B595, U3 Pollin_DCF1, U4 TPIC6B595, U5 WeMos_D1_mini, U6 TPIC6B595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

Commit message: First version of complete board
Parts:
- added H1, H2, H3, H4: MountingHole, MountingHole:MountingHole_4.3mm_M4, symbol Mechanical:MountingHole
- U3: footprint Connector_PinSocket_2.54mm:PinSocket_1x04_P2.54mm_Horizontal -> Connector_PinSocket_2.54mm:PinSocket_1x04_P2.54mm_Vertical
Connections:
- net U8-D7: now reaches N4.0, U8.17 (DRAIN7)
- net U7-D6: now reaches N4.1, U7.16 (DRAIN6)
- net U7-D7: now reaches N4.2, U7.17 (DRAIN7)
- net U8-D0: now reaches N4.3, U8.4 (DRAIN0)
- net U8-D1: now reaches N4.4, U8.5 (DRAIN1)
- net U8-D2: now reaches N4.5, U8.6 (DRAIN2)
- net U8-D3: now reaches N4.6, U8.7 (DRAIN3)
- net U8-D4: now reaches N4.7, U8.14 (DRAIN4)
- net U8-D5: now reaches N4.8, U8.15 (DRAIN5)
- net U8-D6: now reaches N4.9, U8.16 (DRAIN6)
- net N4-A: now reaches N4.A, R6.2
- net at U5.4 (SCK/D5): now also U1.13; no longer U1.5
- net at U5.6 (MOSI/D7): now also U1.11; no longer U1.3
- net at R4.1, U5.7 (CS/D8): now also U1.9; no longer U1.1
- net U6-D3: now reaches N2.0, U6.7 (DRAIN3)
- net U4-D2: now reaches N2.1, U4.6 (DRAIN2)
- net U4-D3: now reaches N2.2, U4.7 (DRAIN3)
- net U4-D4: now reaches N2.3, U4.14 (DRAIN4)
- net U4-D5: now reaches N2.4, U4.15 (DRAIN5)
- net U4-D6: now reaches N2.5, U4.16 (DRAIN6)
- net U4-D7: now reaches N2.6, U4.17 (DRAIN7)
- net U6-D0: now reaches N2.7, U6.4 (DRAIN0)
- net U6-D1: now reaches N2.8, U6.5 (DRAIN1)
- net U6-D2: now reaches N2.9, U6.6 (DRAIN2)
- net N2-A: now reaches N2.A, R3.2
- net U11-D3: now reaches N6.0, U11.7 (DRAIN3)
- net U10-D2: now reaches N6.1, U10.6 (DRAIN2)
- net U10-D3: now reaches N6.2, U10.7 (DRAIN3)
- net U10-D4: now reaches N6.3, U10.14 (DRAIN4)
- net U10-D5: now reaches N6.4, U10.15 (DRAIN5)
- net U10-D6: now reaches N6.5, U10.16 (DRAIN6)
- net U10-D7: now reaches N6.6, U10.17 (DRAIN7)
- net U11-D0: now reaches N6.7, U11.4 (DRAIN0)
- net U11-D1: now reaches N6.8, U11.5 (DRAIN1)
- net U11-D2: now reaches N6.9, U11.6 (DRAIN2)
- net N6-A: now reaches N6.A, R8.2
- net at U10.12 (RCLK), U11.12 (RCLK), U2.12 (RCLK)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: now also U1.4; no longer U1.10
- net at U10.13 (SRCK), U11.13 (SRCK), U2.13 (SRCK)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: now also U1.2; no longer U1.8
- net U6-D4: now reaches N3.1, U6.14 (DRAIN4)
- net U6-D5: now reaches N3.2, U6.15 (DRAIN5)
- net U6-D6: now reaches N3.3, U6.16 (DRAIN6)
- net U6-D7: now reaches N3.4, U6.17 (DRAIN7)
- net at U1.6: now also U2.3 (SER_IN); no longer U1.9
- net U2-D4: now reaches N1.5, U2.14 (DRAIN4)
- net U2-D5: now reaches N1.6, U2.15 (DRAIN5)
- net U2-D6: now reaches N1.7, U2.16 (DRAIN6)
- net U2-D7: now reaches N1.8, U2.17 (DRAIN7)
- net at U1.12: now also U1.1; no longer U2.3 (SER_IN)
- net U2-D0: now reaches N1.1, U2.4 (DRAIN0)
- net U2-D1: now reaches N1.2, U2.5 (DRAIN1)
- net U2-D2: now reaches N1.3, U2.6 (DRAIN2)
- net U2-D3: now reaches N1.4, U2.7 (DRAIN3)
- net U7-D4: now reaches N3.9, U7.14 (DRAIN4)
- net U7-D5: now reaches N3.0, U7.15 (DRAIN5)
- net U7-D0: now reaches N3.5, U7.4 (DRAIN0)
- net U7-D1: now reaches N3.6, U7.5 (DRAIN1)
- net U7-D2: now reaches N3.7, U7.6 (DRAIN2)
- net U7-D3: now reaches N3.8, U7.7 (DRAIN3)
- net N3-A: now reaches N3.A, R5.2
- net U10-D0: now reaches N5.9, U10.4 (DRAIN0)
- net U10-D1: now reaches N5.0, U10.5 (DRAIN1)
- net U4-D0: now reaches N1.9, U4.4 (DRAIN0)
- net U4-D1: now reaches N1.0, U4.5 (DRAIN1)
- net N1-A: now reaches N1.A, R1.2
- net U9-D0: now reaches N5.1, U9.4 (DRAIN0)
- net U9-D1: now reaches N5.2, U9.5 (DRAIN1)
- net U9-D2: now reaches N5.3, U9.6 (DRAIN2)
- net U9-D3: now reaches N5.4, U9.7 (DRAIN3)
- net U9-D4: now reaches N5.5, U9.14 (DRAIN4)
- net U9-D5: now reaches N5.6, U9.15 (DRAIN5)
- net U9-D6: now reaches N5.7, U9.16 (DRAIN6)
- net U9-D7: now reaches N5.8, U9.17 (DRAIN7)
- net N5-A: now reaches N5.A, R7.2
- new net: U1.3, U1.8
- new net: U1.10, U1.5
Other:
- moved on the sheet: U1A, U1B, U1C, U1D, U1E, U1F
